Commit message: feat : can learn seds and send torque coomands

File: hls/zobotics/robot.urdf (robot description, URDF)
Before this commit: robot zobotics, 5 links, 4 joints
Joints:
- joint servo2shaft2: limit lower=-0.43 upper=2.20 effort=2.5 velocity=60 -> lower=-1.40 upper=2.75 effort=2.5 velocity=60

Commit message: feat : last commit maison abandonnée

File: hls/zobotics/robot.urdf (robot description, URDF)
Before this commit: robot zobotics, 5 links, 4 joints
Joints:
- joint servo2shaft3: limit lower=-2.0 upper=2.36 effort=2.5 velocity=60 -> lower=-2.20 upper=3.34 effort=2.5 velocity=60
